File: HW2.X/PCB/PCB.brd (EAGLE design)
At the start: 50 x 50 mm, 22 parts

Commit message: PCB Update
Parts:
- moved LED1 6.35 mm to (33.7, 3.17)
- moved R3 2.54 mm to (48.3, 8.26)
- moved U$1 1.00 mm to (24.4, 47.3), turned to 180 degrees
- moved R4 0.63 mm to (10.2, 14.6)
Routing:
- net +3V3: track 0.00 -> 134.1 mm
- net +5V: track 0.00 -> 96.7 mm
- net MCLR: track 0.00 -> 70.1 mm, vias 0 -> 3
- net USBID: track 0.00 -> 57.6 mm, vias 0 -> 2
- net A4: track 0.00 -> 46.5 mm, vias 0 -> 2
- net B4: track 0.00 -> 41.1 mm, vias 0 -> 1
- net D-: track 0.00 -> 38.5 mm
- net B7: track 0.00 -> 28.7 mm
- net D+: track 0.00 -> 25.8 mm
- net B9: track 0.00 -> 25.5 mm
- net PEGC1: track 0.00 -> 24.7 mm
- net PEGD1: track 0.00 -> 24.7 mm
- net B8: track 0.00 -> 24.5 mm
- net A0: track 0.00 -> 23.2 mm
- net A1: track 0.00 -> 23.2 mm
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- added copper zone on layer 16, net GND

Commit message: Upload dru file
Routing:
- net VBUS: track 17.8 -> 16.1 mm
Changed lines of the file:
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@@
 <vertex x="0" y="0"/>
 </polygon>
+<wire x1="25.7175" y1="47.3075" x2="30.48" y2="38.1" width="0" layer="19" extent="1-1"/>
 </signal>
 <signal name="N$1">
@@
 <wire x1="36.5125" y1="43.4975" x2="45.4025" y2="43.4975" width="0.4064" layer="16"/>
 <wire x1="45.4025" y1="43.4975" x2="46.99" y2="41.91" width="0.4064" layer="16"/>
-<wire x1="46.99" y1="41.91" x2="46.99" y2="41.56" width="0.4064" layer="16"/>
-<wire x1="46.99" y1="41.56" x2="46.05" y2="40.62" width="0.4064" layer="16"/>
+<wire x1="46.99" y1="41.91" x2="46.05" y2="40.62" width="0" layer="19" extent="1-16"/>
 </signal>
 <signal name="MCLR">
